File: RasPi-BplusHAT.brd (EAGLE design)
At the start: 65 x 56 mm, 10 parts, among them K1 PIN20X2

Commit message: Fixes
Parts:
- renumbered S1 to GPIO27, S2 to GPIO17, S3 to GPIO18, S4 to GPIO25
Other:
- board text added: "BKLED (GPIO22)"
