File: RasPi-BplusHAT.sch (EAGLE design)
At the start: 10 parts, among them K1 PIN20X2

Commit message: Fixes
Parts:
- renumbered S1 to GPIO27, S2 to GPIO17, S3 to GPIO18, S4 to GPIO25
Changed lines of the file:
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@@
 </variantdefs>
 <classes>
-<class number="0" name="default" width="0.3048" drill="0.254">
+<class number="0" name="default" width="0.3048" drill="0.381">
 <clearance class="0" value="0.3048"/>
 </class>
@@
 <part name="GND3" library="supply1" deviceset="GND" device=""/>
 <part name="P+1" library="supply1" deviceset="+5V" device=""/>
-<part name="S1" library="switch-omron" library_urn="urn:adsk.eagle:library:377" deviceset="10-XX" device="" package3d_urn="urn:adsk.eagle:package:27496/1"/>
-<part name="S2" library="switch-omron" library_urn="urn:adsk.eagle:library:377" deviceset="10-XX" device="" package3d_urn="urn:adsk.eagle:package:27496/1"/>
-<part name="S3" library="switch-omron" library_urn="urn:adsk.eagle:library:377" deviceset="10-XX" device="" package3d_urn="urn:adsk.eagle:package:27496/1"/>
-<part name="S4" library="switch-omron" library_urn="urn:adsk.eagle:library:377" deviceset="10-XX" device="" package3d_urn="urn:adsk.eagle:package:27496/1"/>
+<part name="GPIO27" library="switch-omron" library_urn="urn:adsk.eagle:library:377" deviceset="10-XX" device="" package3d_urn="urn:adsk.eagle:package:27496/1"/>
+<part name="GPIO17" library="switch-omron" library_urn="urn:adsk.eagle:library:377" deviceset="10-XX" device="" package3d_urn="urn:adsk.eagle:package:27496/1"/>
+<part name="GPIO18" library="switch-omron" library_urn="urn:adsk.eagle:library:377" deviceset="10-XX" device="" package3d_urn="urn:adsk.eagle:package:27496/1"/>
+<part name="GPIO25" library="switch-omron" library_urn="urn:adsk.eagle:library:377" deviceset="10-XX" device="" package3d_urn="urn:adsk.eagle:package:27496/1"/>
 <part name="REG1" library="resistor" library_urn="urn:adsk.eagle:library:348" deviceset="R-EU_" device="0204/7" package3d_urn="urn:adsk.eagle:package:25945/1" value="10K"/>
 <part name="REG2" library="resistor" library_urn="urn:adsk.eagle:library:348" deviceset="R-EU_" device="0204/7" package3d_urn="urn:adsk.eagle:package:25945/1" value="10K"/>
@@
 <part name="GND4" library="supply1" deviceset="GND" device=""/>
 <part name="GND5" library="supply1" deviceset="GND" device=""/>
-<part name="SV1" library="con-lsta" library_urn="urn:adsk.eagle:library:161" deviceset="FE08-1" device="" package3d_urn="urn:adsk.eagle:package:8194/1"/>
+<part name="SV1" library="con-lsta" deviceset="FE08-1" device="" package3d_urn="urn:adsk.eagle:package:8194/1"/>
 </parts>
 <sheets>
@@
 <attribute name="VALUE" x="63.5" y="185.42" size="1.778" layer="96" rot="R180"/>
 </instance>
-<instance part="S1" gate="1" x="91.44" y="175.26" smashed="yes">
+<instance part="GPIO27" gate="1" x="91.44" y="175.26" smashed="yes">
 <attribute name="NAME" x="85.09" y="172.72" size="1.778" layer="95" rot="R90"/>
 <attribute name="VALUE" x="87.63" y="178.435" size="1.778" layer="96" rot="R90"/>
 </instance>
-<instance part="S2" gate="1" x="91.44" y="147.32" smashed="yes">
+<instance part="GPIO17" gate="1" x="91.44" y="147.32" smashed="yes">
 <attribute name="NAME" x="85.09" y="144.78" size="1.778" layer="95" rot="R90"/>
 <attribute name="VALUE" x="87.63" y="150.495" size="1.778" layer="96" rot="R90"/>
 </instance>
-<instance part="S3" gate="1" x="91.44" y="119.38" smashed="yes">
+<instance part="GPIO18" gate="1" x="91.44" y="119.38" smashed="yes">
 <attribute name="NAME" x="85.09" y="116.84" size="1.778" layer="95" rot="R90"/>
 <attribute name="VALUE" x="87.63" y="122.555" size="1.778" layer="96" rot="R90"/>
 </instance>
-<instance part="S4" gate="1" x="91.44" y="200.66" smashed="yes">
+<instance part="GPIO25" gate="1" x="91.44" y="200.66" smashed="yes">
 <attribute name="NAME" x="85.09" y="198.12" size="1.778" layer="95" rot="R90"/>
 <attribute name="VALUE" x="87.63" y="203.835" size="1.778" layer="96" rot="R90"/>
@@
 </segment>
 <segment>
-<pinref part="S3" gate="1" pin="P1"/>
+<pinref part="GPIO18" gate="1" pin="P1"/>
 <pinref part="GND1" gate="1" pin="GND"/>
 <wire x1="93.98" y1="114.3" x2="93.98" y2="111.76" width="0.1524" layer="91"/>
@@
 </segment>
 <segment>
-<pinref part="S2" gate="1" pin="P1"/>
+<pinref part="GPIO17" gate="1" pin="P1"/>
 <pinref part="GND2" gate="1" pin="GND"/>
 <wire x1="93.98" y1="142.24" x2="93.98" y2="139.7" width="0.1524" layer="91"/>
@@
 </segment>
 <segment>
-<pinref part="S1" gate="1" pin="P1"/>
+<pinref part="GPIO27" gate="1" pin="P1"/>
 <pinref part="GND4" gate="1" pin="GND"/>
 <wire x1="93.98" y1="170.18" x2="101.6" y2="170.18" width="0.1524" layer="91"/>
 </segment>
 <segment>
-<pinref part="S4" gate="1" pin="P1"/>
+<pinref part="GPIO25" gate="1" pin="P1"/>
 <pinref part="GND5" gate="1" pin="GND"/>
 <wire x1="93.98" y1="195.58" x2="101.6" y2="195.58" width="0.1524" layer="91"/>
@@
 <net name="N$1" class="0">
 <segment>
-<pinref part="S4" gate="1" pin="S1"/>
+<pinref part="GPIO25" gate="1" pin="S1"/>
 <pinref part="REG1" gate="G$1" pin="2"/>
 <wire x1="104.14" y1="205.74" x2="93.98" y2="205.74" width="0.1524" layer="91"/>
@@
 <net name="N$2" class="0">
 <segment>
-<pinref part="S1" gate="1" pin="S1"/>
+<pinref part="GPIO27" gate="1" pin="S1"/>
 <pinref part="REG2" gate="G$1" pin="2"/>
 <wire x1="104.14" y1="180.34" x2="93.98" y2="180.34" width="0.1524" layer="91"/>
@@
 <net name="N$3" class="0">
 <segment>
-<pinref part="S2" gate="1" pin="S1"/>
+<pinref part="GPIO17" gate="1" pin="S1"/>
 <pinref part="REG3" gate="G$1" pin="2"/>
 <wire x1="104.14" y1="152.4" x2="93.98" y2="152.4" width="0.1524" layer="91"/>
@@
 <net name="N$4" class="0">
 <segment>
-<pinref part="S3" gate="1" pin="S1"/>
+<pinref part="GPIO18" gate="1" pin="S1"/>
 <pinref part="REG4" gate="G$1" pin="2"/>
 <wire x1="104.14" y1="124.46" x2="93.98" y2="124.46" width="0.1524" layer="91"/>
@@
 <net name="BUTTON3" class="0">
 <segment>
-<pinref part="S1" gate="1" pin="S"/>
+<pinref part="GPIO27" gate="1" pin="S"/>
 <wire x1="91.44" y1="180.34" x2="91.44" y2="185.42" width="0.1524" layer="91"/>
 <label x="91.44" y="185.42" size="1.778" layer="95"/>
@@
 <net name="BUTTON4" class="0">
 <segment>
-<pinref part="S4" gate="1" pin="S"/>
+<pinref part="GPIO25" gate="1" pin="S"/>
 <wire x1="91.44" y1="205.74" x2="91.44" y2="210.82" width="0.1524" layer="91"/>
 <label x="91.44" y="210.82" size="1.778" layer="95"/>
@@
 <net name="BUTTON2" class="0">
 <segment>
-<pinref part="S2" gate="1" pin="S"/>
+<pinref part="GPIO17" gate="1" pin="S"/>
 <wire x1="91.44" y1="152.4" x2="91.44" y2="157.48" width="0.1524" layer="91"/>
 <label x="91.44" y="157.48" size="1.778" layer="95"/>
@@
 <net name="BUTTON1" class="0">
 <segment>
-<pinref part="S3" gate="1" pin="S"/>
+<pinref part="GPIO18" gate="1" pin="S"/>
 <wire x1="91.44" y1="124.46" x2="91.44" y2="129.54" width="0.1524" layer="91"/>
 <label x="91.44" y="129.54" size="1.778" layer="95"/>
